File: LOGIC-SHIELD/HARDWARE/REV A/SINGLE/TH.kicad_pcb (KiCad board)
At the start: 2 copper layers, 56.9 x 53.1 mm, 13 parts, among them P1 CONN_02X08, P2 CONN_02X08, P3 CONN_01X08, P4 CONN_01X06, P5 CONN_01X10, P6 CONN_01X08, P7 CONN_02X08, U1 SST39VF010-70-4C-NHE

Commit message: added some repos, changed names of others
Parts:
- removed U1: SST39VF010-70-4C-NHE, MOD:PLCC-32
