File: T85DUINO/HARDWARE/REV B/SINGLE/TH.sch (KiCad schematic (older format))
At the start: 13 parts, among them P1 USB_OTG, P2 ICSP, SW1 Push_SW, U1 ATTINY85-P

Commit message: rev b and license
Parts:
- added R3: 1.5K, Resistors_THT:Resistor_Horizontal_RM7mm, symbol R
Connections:
- net VCC: now also R3.1
- net at P1.3 (D+), R2.2: now also R3.2
Other:
- moved on the sheet: P1
Changed lines of the file:
@@
 $EndDescr
 $Comp
-L GND #PWR01
+L GND #PWR1
 U 1 1 5AB9F53C
-P 2300 4250
-F 0 "#PWR01" H 2300 4000 50  0001 C CNN
-F 1 "GND" H 2300 4100 50  0000 C CNN
-F 2 "" H 2300 4250 50  0000 C CNN
-F 3 "" H 2300 4250 50  0000 C CNN
-	1    2300 4250
+P 1950 4250
+F 0 "#PWR1" H 1950 4000 50  0001 C CNN
+F 1 "GND" H 1950 4100 50  0000 C CNN
+F 2 "" H 1950 4250 50  0000 C CNN
+F 3 "" H 1950 4250 50  0000 C CNN
+	1    1950 4250
 	-1   0    0    -1
 $EndComp
 Wire Wire Line
-	2300 4250 2300 4150
-$Comp
-L GND #PWR02
+	1950 4250 1950 4150
+$Comp
+L GND #PWR2
 U 1 1 5AB9F5CF
-P 2700 4050
-F 0 "#PWR02" H 2700 3800 50  0001 C CNN
-F 1 "GND" H 2700 3900 50  0000 C CNN
-F 2 "" H 2700 4050 50  0000 C CNN
-F 3 "" H 2700 4050 50  0000 C CNN
-	1    2700 4050
+P 2350 4050
+F 0 "#PWR2" H 2350 3800 50  0001 C CNN
+F 1 "GND" H 2350 3900 50  0000 C CNN
+F 2 "" H 2350 4050 50  0000 C CNN
+F 3 "" H 2350 4050 50  0000 C CNN
+	1    2350 4050
 	-1   0    0    -1
 $EndComp
@@
 $EndComp
 $Comp
-L GND #PWR03
+L GND #PWR10
 U 1 1 5ABA3B72
 P 9050 4100
-F 0 "#PWR03" H 9050 3850 50  0001 C CNN
+F 0 "#PWR10" H 9050 3850 50  0001 C CNN
 F 1 "GND" H 9050 3950 50  0000 C CNN
 F 2 "" H 9050 4100 50  0000 C CNN
@@
 	0    1    -1   0
 $EndComp
-NoConn ~ 2700 3550
-Wire Wire Line
-	2700 3650 2800 3650
-Wire Wire Line
-	2800 3750 2700 3750
+NoConn ~ 2350 3550
+Wire Wire Line
+	2350 3650 2800 3650
+Wire Wire Line
+	2350 3750 2800 3750
 Wire Wire Line
 	3100 3650 3650 3650
@@
 $EndComp
 $Comp
-L GND #PWR04
+L GND #PWR5
 U 1 1 5BE11532
 P 4450 4350
-F 0 "#PWR04" H 4450 4100 50  0001 C CNN
+F 0 "#PWR5" H 4450 4100 50  0001 C CNN
 F 1 "GND" H 4450 4200 50  0000 C CNN
 F 2 "" H 4450 4350 50  0000 C CNN
@@
 	3550 3450 3650 3450
 Wire Wire Line
-	2700 4050 2700 3950
+	2350 4050 2350 3950
 $Comp
 L USB_OTG P1
 U 1 1 5BE11202
-P 2400 3750
-F 0 "P1" V 2725 3625 50  0000 C CNN
-F 1 "USB_OTG" H 2400 3950 50  0000 C CNN
-F 2 "MOD:TE_2172034-1" V 2350 3650 50  0001 C CNN
-F 3 "" V 2350 3650 50  0000 C CNN
-	1    2400 3750
+P 2050 3750
+F 0 "P1" V 2375 3625 50  0000 C CNN
+F 1 "USB_OTG" H 2050 3950 50  0000 C CNN
+F 2 "MOD:TE_2172034-1" V 2000 3650 50  0001 C CNN
+F 3 "" V 2000 3650 50  0000 C CNN
+	1    2050 3750
 	0    -1   1    0
 $EndComp
@@
 	6650 3850 6350 3850
 $Comp
-L GND #PWR05
+L GND #PWR7
 U 1 1 5BE11D5F
 P 6650 3850
-F 0 "#PWR05" H 6650 3600 50  0001 C CNN
+F 0 "#PWR7" H 6650 3600 50  0001 C CNN
 F 1 "GND" H 6650 3700 50  0000 C CNN
 F 2 "" H 6650 3850 50  0000 C CNN
@@
 $EndComp
 $Comp
-L GND #PWR06
+L GND #PWR4
 U 1 1 5BE125D5
 P 2800 3150
-F 0 "#PWR06" H 2800 2900 50  0001 C CNN
+F 0 "#PWR4" H 2800 2900 50  0001 C CNN
 F 1 "GND" H 2800 3000 50  0000 C CNN
 F 2 "" H 2800 3150 50  0000 C CNN
@@
 MOSI
 $Comp
-L VCC #PWR07
+L VCC #PWR8
 U 1 1 5BE25593
 P 8100 3350
-F 0 "#PWR07" H 8100 3200 50  0001 C CNN
+F 0 "#PWR8" H 8100 3200 50  0001 C CNN
 F 1 "VCC" H 8100 3500 50  0000 C CNN
 F 2 "" H 8100 3350 50  0000 C CNN
@@
 	8100 3350 8100 3450
 $Comp
-L GND #PWR08
+L GND #PWR9
 U 1 1 5BE255E4
 P 8100 3750
-F 0 "#PWR08" H 8100 3500 50  0001 C CNN
+F 0 "#PWR9" H 8100 3500 50  0001 C CNN
 F 1 "GND" H 8100 3600 50  0000 C CNN
 F 2 "" H 8100 3750 50  0000 C CNN
@@
 	2800 3150 2700 3150
 $Comp
-L VCC #PWR?
+L VCC #PWR6
 U 1 1 5BE26B74
 P 6650 3350
-F 0 "#PWR?" H 6650 3200 50  0001 C CNN
+F 0 "#PWR6" H 6650 3200 50  0001 C CNN
 F 1 "VCC" H 6650 3500 50  0000 C CNN
 F 2 "" H 6650 3350 50  0000 C CNN
@@
 	1    0    0    -1
 $EndComp
+$Comp
+L R R3
+U 1 1 5BE8B5BE
+P 2700 4000
+F 0 "R3" V 2780 4000 50  0000 C CNN
+F 1 "1.5K" V 2700 4000 50  0000 C CNN
+F 2 "Resistors_THT:Resistor_Horizontal_RM7mm" V 2630 4000 50  0001 C CNN
+F 3 "" H 2700 4000 50  0000 C CNN
+	1    2700 4000
+	1    0    0    1
+$EndComp
+$Comp
+L VCC #PWR3
+U 1 1 5BE8B89E
+P 2700 4250
+F 0 "#PWR3" H 2700 4100 50  0001 C CNN
+F 1 "VCC" H 2700 4400 50  0000 C CNN
+F 2 "" H 2700 4250 50  0000 C CNN
+F 3 "" H 2700 4250 50  0000 C CNN
+	1    2700 4250
+	-1   0    0    1
+$EndComp
+Wire Wire Line
+	2700 4250 2700 4150
+Wire Wire Line
+	2700 3750 2700 3850
+Connection ~ 2700 3750
 $EndSCHEMATC
