File: T85DUINO/HARDWARE/REV B/SINGLE/TH.kicad_pcb (KiCad board)
At the start: 2 copper layers, 34.3 x 26.5 mm, 14 parts, among them P1 USB_OTG, P2 ICSP, SW1 Push_SW, U1 ATTINY85-P

Commit message: rev b and license
Parts:
- added R3: 1.5K, Resistors_THT:Resistor_Horizontal_RM7mm, F.Cu at (133.1, 114.6)
- moved D2 3.21 mm to (129.3, 110.6), turned to 180 degrees
- moved C1 2.69 mm to (135.8, 111.6), turned to 180 degrees
Routing:
- net VCC: track 33.4 -> 38.2 mm
- net Net-(D2-Pad2): track 5.75 -> 3.80 mm
- net MISO: track 33.2 -> 34.2 mm
- net Net-(P1-Pad2): track 22.5 -> 23.2 mm
Other:
- board text added: "CDM R:B 11-11-18"
- board text added: "PB1 PB0"
- board text added: "PB2"
- board text added: "RST"
- board text removed: "CDM R:A 11-6-18"

Commit message: updated XMAS
Parts:
- P1: footprint MOD:TE_2172034-1 -> MOD:USB_MINI_B_TH
- R3: footprint Resistors_THT:Resistor_Horizontal_RM7mm -> MOD:Resistor_Horizontal_RM7mm
Routing:
- net GND: track 13.3 -> 7.37 mm
