File: XMAS/HARDWARE/REV B/XMAS.sch (KiCad schematic (older format))
At the start: 31 parts, among them P1 ICSP, SW1 Push_SW, U1 MCP6541T-I/LT, U2 ATTINY24A-M

Commit message: updated XMAS
Parts:
- C1: value C -> 0.1uF
- SW1: footprint MOD:JS102011JAQN_NO_DRILL -> MOD:JS102011JAQN_Handsoldering
- U1: value MCP6541T-I/LT -> MCP6541R-I/LT
Other:
- note added: "SLIDE SW"
Changed lines of the file:
@@
 LIBS:contrib
 LIBS:valves
-LIBS:MCP6541T-I_LT
-LIBS:push_sw
 LIBS:XMAS-cache
 EELAYER 25 0
@@
 encoding utf-8
 Sheet 1 1
-Title ""
-Date ""
-Rev ""
-Comp ""
+Title "Christmas Ornament"
+Date "2018-11-24"
+Rev "B"
+Comp "Thunkit Electronics"
 Comment1 ""
 Comment2 ""
@@
 P 5950 3250
 F 0 "U1" H 5950 3250 47  0000 C CNN
-F 1 "MCP6541T-I/LT" H 6000 2600 47  0000 C CNN
+F 1 "MCP6541R-I/LT" H 6000 2600 47  0000 C CNN
 F 2 "TO_SOT_Packages_SMD:SOT-23-5" H 5950 3250 47  0001 C CNN
 F 3 "" H 5950 3250 47  0001 C CNN
@@
 P 7450 3600
 F 0 "C1" H 7475 3700 50  0000 L CNN
-F 1 "C" H 7475 3500 50  0000 L CNN
+F 1 "0.1uF" H 7475 3500 50  0000 L CNN
 F 2 "Capacitors_SMD:C_0603" H 7488 3450 50  0001 C CNN
 F 3 "" H 7450 3600 50  0000 C CNN
 	1    7450 3600
-	1    0    0    -1
+	-1   0    0    -1
 $EndComp
 $Comp
@@
 F 0 "U2" H 7650 4300 50  0000 C CNN
 F 1 "ATTINY24A-M" H 9200 2800 50  0000 C CNN
-F 2 "Housings_DFN_QFN:QFN-20-1EP_4x4mm_Pitch0.5mm" H 8500 2600 50  0000 C CIN
+F 2 "Housings_DFN_QFN:QFN-20-1EP_4x4mm_Pitch0.5mm" H 8500 2600 50  0001 C CIN
 F 3 "" H 8500 3550 50  0000 C CNN
 	1    8500 3550
@@
 F 0 "SW1" V 3850 3250 47  0000 C CNN
 F 1 "Push_SW" H 3860 3480 47  0001 C CNN
-F 2 "MOD:JS102011JAQN_NO_DRILL" H 3850 3500 47  0001 C CNN
+F 2 "MOD:JS102011JAQN_Handsoldering" H 3850 3500 47  0001 C CNN
 F 3 "" H 3850 3500 47  0001 C CNN
 	1    3850 3500
@@
 Wire Wire Line
 	3000 2700 3000 3200
+Text Notes 4050 3650 0    60   ~ 0
+SLIDE SW
 $EndSCHEMATC
