File: MAKIT-THT/HARDWARE/REV C/SINGLE/TH.sch (KiCad schematic (older format))
At the start: 27 parts, among them P1 USB_A, P2 BARREL_JACK, P3 CONN_01X08, P4 CONN_01X06, P5 CONN_01X10, P6 CONN_01X08, P7 ICSP, SW1 Push_SW, U1 LM7805CT, U2 MCP2221A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

Commit message: updated vreg
Parts:
- U4: value L78L33 -> 3.3V Reg.
Changed lines of the file:
@@
 P 4450 6300
 F 0 "U4" H 4250 6500 50  0000 C CNN
-F 1 "L78L33" H 4450 6500 50  0000 L CNN
+F 1 "3.3V Reg." H 4450 6500 50  0000 L CNN
 F 2 "TO_SOT_Packages_THT:TO-92_Inline_Wide" H 4450 6400 50  0001 C CIN
 F 3 "" H 4450 6300 50  0000 C CNN
